Commit message: Update model sigmaban urdf

File: newFake/sigmaban.urdf (robot description, URDF)
Before this commit: robot URDF, 26 links, 25 joints
Links:
- removed link camera_link
- removed link head_pitch_link
- removed link head_yaw_link
- removed link left_ankle_pitch_link
- removed link left_ankle_roll_link
- removed link left_arm_tip_link
- removed link left_elbow_link
- removed link left_foot_tip_link
- removed link left_hip_pitch_link
- removed link left_hip_roll_link
- removed link left_hip_yaw_link
- removed link left_knee_link
- removed link left_shoulder_pitch_link
- removed link left_shoulder_roll_link
- removed link right_ankle_pitch_link
- removed link right_ankle_roll_link
- removed link right_arm_tip_link
- removed link right_elbow_link
- removed link right_foot_tip_link
- removed link right_hip_pitch_link
- removed link right_hip_roll_link
- removed link right_hip_yaw_link
- removed link right_knee_link
- removed link right_shoulder_pitch_link
- removed link right_shoulder_roll_link
- removed link trunk_link
- added link camera, mass 0
- added link head_pitch, mass 0.081452; collision box size=0.0354 0.0504 0.0353; visual mesh filename=package://urdf/2315e68be0ea2e6e80f047b6547c6a9dfbdc80f4.stl
- added link head_yaw, mass 0.028492; collision box size=0.0018 0.0298 0.0238; collision box size=0.0018 0.0298 0.0238
- added link left_ankle_pitch, mass 0.288805; collision box size=0.04 0.0609 0.0408; collision box size=0.04 0.0609 0.0408
- added link left_ankle_roll, mass 0.196741; collision box size=0.0018 0.0298 0.0298; collision box size=0.0018 0.0298 0.0298
- added link left_arm_tip, mass 0
- added link left_elbow, mass 0.136991; collision box size=0.0354 0.0018 0.0912; collision box size=0.0354 0.0374 0.0018
- added link left_foot_tip, mass 0
- added link left_hip_pitch, mass 0.195989; collision box size=0.0018 0.0298 0.0737; collision box size=0.0018 0.0298 0.0737
- added link left_hip_roll, mass 0.288805; collision box size=0.04 0.0609 0.0408; collision box size=0.04 0.0609 0.0408
- added link left_hip_yaw, mass 0.032317; collision box size=0.0018 0.0298 0.0298; collision box size=0.0018 0.0298 0.0298
- added link left_knee, mass 0.06154; collision box size=0.1378 0.0278 0.0018; collision box size=0.1378 0.0278 0.0018
- added link left_shoulder_pitch, mass 0.029002; collision box size=0.0018 0.0298 0.0248; collision box size=0.0018 0.0298 0.0248
- added link left_shoulder_roll, mass 0.150302; collision box size=0.0018 0.0298 0.0298; collision box size=0.0018 0.0298 0.0298
- added link right_ankle_pitch, mass 0.288805; collision box size=0.04 0.0609 0.0408; collision box size=0.04 0.0609 0.0408
- added link right_ankle_roll, mass 0.196741; collision box size=0.0018 0.0298 0.0298; collision box size=0.0018 0.0298 0.0298
- added link right_arm_tip, mass 0
- added link right_elbow, mass 0.136991; collision box size=0.0354 0.0018 0.0912; collision box size=0.0354 0.0374 0.0018
- added link right_foot_tip, mass 0
- added link right_hip_pitch, mass 0.195989; collision box size=0.0018 0.0298 0.0737; collision box size=0.0018 0.0298 0.0737
- added link right_hip_roll, mass 0.288805; collision box size=0.04 0.0609 0.0408; collision box size=0.04 0.0609 0.0408
- added link right_hip_yaw, mass 0.032317; collision box size=0.0018 0.0298 0.0298; collision box size=0.0018 0.0298 0.0298
- added link right_knee, mass 0.06154; collision box size=0.1378 0.0278 0.0018; collision box size=0.1378 0.0278 0.0018
- added link right_shoulder_pitch, mass 0.029002; collision box size=0.0018 0.0298 0.0248; collision box size=0.0018 0.0298 0.0248
- added link right_shoulder_roll, mass 0.150302; collision box size=0.0018 0.0298 0.0298; collision box size=0.0018 0.0298 0.0298
- added link trunk, mass 1.37255; collision box size=0.0354 0.0504 0.0353; collision box size=0.0354 0.0504 0.0353
Joints:
- removed joint camera_fixed
- removed joint left_arm_tip_fixed
- removed joint left_foot_tip_fixed
- removed joint right_arm_tip_fixed
- removed joint right_foot_tip_fixed
- added joint camera: type fixed, parent head_pitch, child camera, origin xyz=0.01 1.59872e-17 0.062 rpy=0 -0 0, axis 0 0 0
- added joint left_arm_tip: type fixed, parent left_elbow, child left_arm_tip, origin xyz=-0.0108 3.78104e-09 -0.1297 rpy=4.37114e-08 -4.37114e-08 1.74846e-07, axis 0 0 0
- added joint left_foot_tip: type fixed, parent left_ankle_roll, child left_foot_tip, origin xyz=2.66639e-09 -5.33279e-09 -0.061 rpy=-8.74228e-08 -4.37114e-08 4.37114e-08, axis 0 0 0
- added joint right_arm_tip: type fixed, parent right_elbow, child right_arm_tip, origin xyz=-0.0108 4.7252e-09 -0.1297 rpy=4.37114e-08 -4.37114e-08 8.74228e-08, axis 0 0 0
- added joint right_foot_tip: type fixed, parent right_ankle_roll, child right_foot_tip, origin xyz=2.66639e-09 -5.33279e-09 -0.061 rpy=-8.74228e-08 -4.37114e-08 4.37114e-08, axis 0 0 0
- joint head_pitch: child head_pitch_link -> head_pitch; limit (none) -> lower=-3.14159 upper=3.14159 effort=2.8 velocity=12; origin xyz=0 0 0.046 rpy=1.3514E-14 9.7219E-31 -0.0010782 -> xyz=0 0 0.04575 rpy=0 -0 0; parent head_yaw_link -> head_yaw; type continuous -> revolute
- joint head_yaw: child head_yaw_link -> head_yaw; limit (none) -> lower=-3.14159 upper=3.14159 effort=2.8 velocity=12; origin xyz=0.02687 -2.9396E-05 0.1525 rpy=-1.3173E-14 1.4204E-17 -2.1314E-14 -> xyz=0.018 0 0.16725 rpy=0 -0 0; parent trunk_link -> trunk; type continuous -> revolute
- joint left_ankle_pitch: child left_ankle_pitch_link -> left_ankle_pitch; limit (none) -> lower=-3.14159 upper=3.14159 effort=6.4 velocity=14; origin xyz=0 0 -0.105 rpy=0 0 0 -> xyz=-4.5897e-09 -9.17939e-09 -0.105 rpy=0 -7.57953e-26 -6.61744e-24; parent left_knee_link -> left_knee; type continuous -> revolute
- joint left_ankle_roll: child left_ankle_roll_link -> left_ankle_roll; limit (none) -> lower=-3.14159 upper=3.14159 effort=6.4 velocity=14; origin xyz=0 0 0 rpy=0 0 0 -> xyz=0 0 0 rpy=1.83244e-25 6.61744e-24 -6.61744e-24; parent left_ankle_pitch_link -> left_ankle_pitch; type continuous -> revolute
- joint left_elbow: child left_elbow_link -> left_elbow; limit (none) -> lower=-3.14159 upper=3.14159 effort=2.8 velocity=12; origin xyz=0.0110000000000031 -0.00100697698549028 -0.0954999266876771 rpy=-7.30574676925524E-05 -1.09269268670997E-16 7.98293607992287E-21 -> xyz=0.0122 5.77427e-09 -0.1077 rpy=0 -1.75549e-24 0; parent left_shoulder_roll_link -> left_shoulder_roll; type continuous -> revolute
- joint left_hip_pitch: child left_hip_pitch_link -> left_hip_pitch; limit (none) -> lower=-3.14159 upper=3.14159 effort=6.4 velocity=14; origin xyz=0 0 0 rpy=0 0 0 -> xyz=0 0 0 rpy=0 -1.85711e-32 0; parent left_hip_roll_link -> left_hip_roll; type continuous -> revolute
- joint left_hip_roll: child left_hip_roll_link -> left_hip_roll; limit (none) -> lower=-3.14159 upper=3.14159 effort=6.4 velocity=14; origin xyz=-0.0004 0 -0.0505 rpy=7.3057E-05 -6.6174E-24 -0.00054721 -> xyz=8.17369e-34 6.67434e-18 -0.0545 rpy=-1.05083e-32 -0 0; parent left_hip_yaw_link -> left_hip_yaw; type continuous -> revolute
- joint left_hip_yaw: child left_hip_yaw_link -> left_hip_yaw; limit (none) -> lower=-3.14159 upper=3.14159 effort=6.4 velocity=14; origin xyz=0.011127 0.046361 0.0105 rpy=-1.5148E-15 8.2889E-19 -0.00053101 -> xyz=0 0.0465 0.0205 rpy=0 -0 0; parent trunk_link -> trunk; type continuous -> revolute
- joint left_knee: child left_knee_link -> left_knee; limit (none) -> lower=-3.14159 upper=3.14159 effort=6.4 velocity=14; origin xyz=0 0 -0.09375 rpy=0 0 0 -> xyz=3.41936e-16 -8.30516e-09 -0.095 rpy=0 -0 -6.61744e-24; parent left_hip_pitch_link -> left_hip_pitch; type continuous -> revolute
- joint left_shoulder_pitch: child left_shoulder_pitch_link -> left_shoulder_pitch; limit (none) -> lower=-3.14159 upper=3.14159 effort=2.8 velocity=12; origin xyz=0.0111273159824835 0.0463607067979427 0.141000000000005 rpy=4.91888973129517E-16 6.34190653024847E-17 -0.00107822069516516 -> xyz=0 0.0465 0.1585 rpy=0 -0 0; parent trunk_link -> trunk; type continuous -> revolute
- joint left_shoulder_roll: child left_shoulder_roll_link -> left_shoulder_roll; limit (none) -> lower=-3.14159 upper=3.14159 effort=2.8 velocity=12; origin xyz=0 0.046 0 rpy=7.30574676925163E-05 -6.34190653024847E-17 7.52316386533968E-37 -> xyz=1.61058e-17 0.04675 -1.03806e-17 rpy=4.40543e-25 -3.9443e-31 1.32349e-23; parent left_shoulder_pitch_link -> left_shoulder_pitch; type continuous -> revolute
- joint right_ankle_pitch: child right_ankle_pitch_link -> right_ankle_pitch; limit (none) -> lower=-3.14159 upper=3.14159 effort=6.4 velocity=14; origin xyz=0 0 -0.105 rpy=0 0 -0.0010782 -> xyz=-4.5897e-09 -9.17939e-09 -0.105 rpy=0 -7.57953e-26 -6.61744e-24; parent right_knee_link -> right_knee; type continuous -> revolute
- joint right_ankle_roll: child right_ankle_roll_link -> right_ankle_roll; limit (none) -> lower=-3.14159 upper=3.14159 effort=6.4 velocity=14; origin xyz=0 0 0 rpy=0 0 0 -> xyz=0 0 0 rpy=1.83244e-25 6.61744e-24 -6.61744e-24; parent right_ankle_pitch_link -> right_ankle_pitch; type continuous -> revolute
- joint right_elbow: child right_elbow_link -> right_elbow; limit (none) -> lower=-3.14159 upper=3.14159 effort=2.8 velocity=12; origin xyz=0.0110010643036779 0.000988138993373119 -0.0955000008665828 rpy=-8.49201152241599E-11 7.87720137245097E-08 -0.00107822069514385 -> xyz=0.0122 4.70772e-09 -0.1077 rpy=0 -5.47945e-24 1.32349e-23; parent right_shoulder_roll_link -> right_shoulder_roll; type continuous -> revolute
- joint right_hip_pitch: child right_hip_pitch_link -> right_hip_pitch; limit (none) -> lower=-3.14159 upper=3.14159 effort=6.4 velocity=14; origin xyz=0 0 0 rpy=0 0 0 -> xyz=0 0 0 rpy=0 -1.85711e-32 0; parent right_hip_roll_link -> right_hip_roll; type continuous -> revolute
- joint right_hip_roll: child right_hip_roll_link -> right_hip_roll; limit (none) -> lower=-3.14159 upper=3.14159 effort=6.4 velocity=14; origin xyz=-0.000399999940109093 0 -0.0505000000000031 rpy=7.30574676945229E-05 -6.61744488276427E-24 -0.000547209476051885 -> xyz=8.17369e-34 6.67434e-18 -0.0545 rpy=-1.05083e-32 -0 0; parent right_hip_yaw_link -> right_hip_yaw; type continuous -> revolute
- joint right_hip_yaw: child right_hip_yaw_link -> right_hip_yaw; limit (none) -> lower=-3.14159 upper=3.14159 effort=6.4 velocity=14; origin xyz=0.0111273159824857 -0.0463847022119938 0.0105000000000006 rpy=-1.51475240770665E-15 8.28887913337337E-19 -0.000531011219113274 -> xyz=0 -0.0465 0.0205 rpy=0 -0 0; parent trunk_link -> trunk; type continuous -> revolute
- joint right_knee: child right_knee_link -> right_knee; limit (none) -> lower=-3.14159 upper=3.14159 effort=6.4 velocity=14; origin xyz=0 0 -0.0937499999999984 rpy=0 0 0.00107822069805326 -> xyz=3.41936e-16 -8.30516e-09 -0.095 rpy=0 -0 -6.61744e-24; parent right_hip_pitch_link -> right_hip_pitch; type continuous -> revolute
- joint right_shoulder_pitch: child right_shoulder_pitch_link -> right_shoulder_pitch; limit (none) -> lower=-3.14159 upper=3.14159 effort=2.8 velocity=12; origin xyz=0.0111273159824815 -0.0463847022119884 0.141000000000006 rpy=4.91888973129517E-16 6.34190653024847E-17 -0.00107822069516516 -> xyz=0 -0.0465 0.1585 rpy=0 -0 0; parent trunk_link -> trunk; type continuous -> revolute
- joint right_shoulder_roll: child right_shoulder_roll_link -> right_shoulder_roll; limit (none) -> lower=-3.14159 upper=3.14159 effort=2.8 velocity=12; origin xyz=0 -0.046 0 rpy=-1.3665338392116E-14 -7.87720585415642E-08 0.00107822069514385 -> xyz=-1.03806e-17 -0.04675 -1.03806e-17 rpy=-9.8608e-32 -0 -9.86076e-32; parent right_shoulder_pitch_link -> right_shoulder_pitch; type continuous -> revolute
