Commit message: django camera angular calibration

File: django/django.urdf (robot description, URDF)
Before this commit: robot metabot, 26 links, 25 joints
Joints:
- joint camera: origin xyz=0.01 1.59872e-17 0.062 rpy=0 -0 0 -> xyz=0.01 1.59872e-17 0.062 rpy=0 0.058 -0.035

Commit message: Fixing urdf of django

File: django/django.urdf (robot description, URDF)
Before this commit: robot metabot, 26 links, 25 joints
Joints:
- joint camera: origin xyz=0.01 1.59872e-17 0.062 rpy=0 0.058 -0.035 -> xyz=0.01 1.59872e-17 0.062 rpy=0 0 0
