Commit message: save

File: tom/tom.urdf (robot description, URDF)
Before this commit: robot metabot, 26 links, 25 joints
Joints:
- joint camera: origin xyz=0.01 1.59872e-17 0.062 rpy=0 -0 0 -> xyz=0.01 1.59872e-17 0.062 rpy=0 -0.07 0.0

Commit message: Tom env (wip)

File: tom/tom.urdf (robot description, URDF)
Before this commit: robot metabot, 26 links, 25 joints
Links:
- link head_yaw: mass 0.028492 -> 0.031552; geometry collision box size=0.0018 0.0298 0.0298; collision box size=0.0018 0.0298 0.0298
- link left_elbow: mass 0.158411 -> 0.121691; geometry collision box size=0.0354 0.0018 0.0412; collision box size=0.0354 0.0374 0.0018
- link left_hip_pitch: mass 0.239475 -> 0.218939; geometry collision box size=0.0018 0.0298 0.1187; collision box size=0.0018 0.0298 0.1187
- link left_knee: mass 0.097444 -> 0.078404; geometry collision box size=0.1728 0.0278 0.0018; collision box size=0.1728 0.0278 0.0018
- link left_shoulder_roll: mass 0.161624 -> 0.141734; geometry collision box size=0.0018 0.0298 0.0298; collision box size=0.0018 0.0298 0.0298
- link right_elbow: mass 0.158411 -> 0.121691; geometry collision box size=0.0354 0.0018 0.0412; collision box size=0.0354 0.0374 0.0018
- link right_hip_pitch: mass 0.239475 -> 0.218939; geometry collision box size=0.0018 0.0298 0.1187; collision box size=0.0018 0.0298 0.1187
- link right_knee: mass 0.097444 -> 0.078404; geometry collision box size=0.1728 0.0278 0.0018; collision box size=0.1728 0.0278 0.0018
- link right_shoulder_roll: mass 0.161624 -> 0.141734; geometry collision box size=0.0018 0.0298 0.0298; collision box size=0.0018 0.0298 0.0298
- link trunk: mass 1.50583 -> 1.59255; geometry collision box size=0.0354 0.0504 0.0353; collision box size=0.0354 0.0504 0.0353
Joints:
- joint camera: origin xyz=0.01 1.59872e-17 0.062 rpy=0 -0.07 0.0 -> xyz=0.01 1.59872e-17 0.062 rpy=0 -0 0
- joint head_pitch: origin xyz=0 0 0.04575 rpy=0 -0 0 -> xyz=0 0 0.05175 rpy=0 -0 0
- joint head_yaw: origin xyz=0.018 0 0.19225 rpy=0 -0 0 -> xyz=0.025873 0 0.16193 rpy=0 -0 0
- joint left_ankle_pitch: origin xyz=-7.86805e-09 -1.57361e-08 -0.18 rpy=0 -7.57953e-26 -6.61744e-24 -> xyz=-6.11959e-09 -1.22392e-08 -0.14 rpy=0 -7.57953e-26 -6.61744e-24
- joint left_arm_tip: origin xyz=-0.0108 6.84083e-09 -0.1997 rpy=4.37114e-08 -4.37114e-08 1.74846e-07 -> xyz=-0.0108 1.59547e-09 -0.0797 rpy=4.37114e-08 -4.37114e-08 1.74846e-07
- joint left_elbow: origin xyz=0.0122 7.3916e-09 -0.1447 rpy=0 -1.75549e-24 0 -> xyz=0.0122 4.55036e-09 -0.0797 rpy=0 -1.75549e-24 0
- joint left_hip_yaw: origin xyz=0 0.0465 0.0205 rpy=0 -0 0 -> xyz=0 0.046375 0.0205 rpy=0 -0 0
- joint left_knee: origin xyz=6.48865e-16 -1.57601e-08 -0.180274 rpy=0 -0 -6.61744e-24 -> xyz=5.03906e-16 -1.22392e-08 -0.14 rpy=0 -0 -6.61744e-24
- joint left_shoulder_pitch: origin xyz=0 0.0465 0.1985 rpy=0 -0 0 -> xyz=0 0.046375 0.159 rpy=0 -0 0
- joint right_ankle_pitch: origin xyz=-7.86805e-09 -1.57361e-08 -0.18 rpy=0 -7.57953e-26 -6.61744e-24 -> xyz=-6.11959e-09 -1.22392e-08 -0.14 rpy=0 -7.57953e-26 -6.61744e-24
- joint right_arm_tip: origin xyz=-0.0108 7.785e-09 -0.1997 rpy=4.37114e-08 -4.37114e-08 8.74228e-08 -> xyz=-0.0108 2.53963e-09 -0.0797 rpy=4.37114e-08 -4.37114e-08 8.74228e-08
- joint right_elbow: origin xyz=0.0122 6.32504e-09 -0.1447 rpy=0 -5.47945e-24 1.32349e-23 -> xyz=0.0122 3.4838e-09 -0.0797 rpy=0 -5.47945e-24 1.32349e-23
- joint right_hip_yaw: origin xyz=0 -0.0465 0.0205 rpy=0 -0 0 -> xyz=0 -0.046375 0.0205 rpy=0 -0 0
- joint right_knee: origin xyz=6.48865e-16 -1.57601e-08 -0.180274 rpy=0 -0 -6.61744e-24 -> xyz=5.03906e-16 -1.22392e-08 -0.14 rpy=0 -0 -6.61744e-24
- joint right_shoulder_pitch: origin xyz=0 -0.0465 0.1985 rpy=0 -0 0 -> xyz=0 -0.046375 0.159 rpy=0 -0 0

Commit message: Tom camera position

File: tom/tom.urdf (robot description, URDF)
Before this commit: robot metabot, 26 links, 25 joints
Links:
- link head_pitch: geometry collision box size=0.0354 0.0504 0.0353; visual mesh filename=package://urdf/ac5b3fd3a7e1b612e3a2bffb9086620de61585c3.stl
Joints:
- joint camera: origin xyz=0.01 1.59872e-17 0.062 rpy=0 -0 0 -> xyz=0.01 1.53988e-17 0.05935 rpy=0 -0 0
