Commit message: chewbacca camera zngular offset calibration

File: chewbacca/chewbacca.urdf (robot description, URDF)
Before this commit: robot metabot, 26 links, 25 joints
Joints:
- joint camera: origin xyz=0.01 1.59872e-17 0.062 rpy=0 -0 0 -> xyz=0.01 1.59872e-17 0.062 rpy=0 -0 -0.083

Commit message: Fixing the model of chewbacca.urdf (removing 4.5 deg in yaw)

File: chewbacca/chewbacca.urdf (robot description, URDF)
Before this commit: robot metabot, 26 links, 25 joints
Joints:
- joint camera: origin xyz=0.01 1.59872e-17 0.062 rpy=0 -0 -0.083 -> xyz=0.01 1.59872e-17 0.062 rpy=0 0 0

Commit message: removing offset in chewbacca.urdf

File: chewbacca/chewbacca.urdf (robot description, URDF)
Before this commit: robot metabot, 26 links, 25 joints
Joints:
- joint camera: origin xyz=0.01 1.59872e-17 0.062 rpy=0 -0 -0.083 -> xyz=0.01 0 0.062 rpy=0 0 0

Commit message: Adding head offsets on tom. Chewbacca has the same urdf than django now. Mowgly had tom's urdf (my bad).

File: chewbacca/chewbacca.urdf (robot description, URDF)
Before this commit: robot metabot, 26 links, 25 joints
Joints:
- joint camera: origin xyz=0.01 0 0.062 rpy=0 0 0 -> xyz=0.01 1.59872e-17 0.062 rpy=0 0 0

File: mowgly/mowgly.urdf (robot description, URDF)
Before this commit: robot metabot, 26 links, 25 joints
Joints:
- joint camera: origin xyz=0.01 1.59872e-17 0.062 rpy=0 0.0 0.0 -> xyz=0.01 1.59872e-17 0.062 rpy=0 0 0
