Commit message: Backuping old sigmaban model + linking all models toward sigmaban.urdf + removing collision and visual fields from sigmaban.urdf

File: common/sigmaban.urdf (robot description, URDF)
Before this commit: robot metabot, 26 links, 25 joints
Links:
- link head_pitch: geometry 
- link head_yaw: geometry 
- link left_ankle_pitch: geometry 
- link left_ankle_roll: geometry 
- link left_elbow: geometry 
- link left_hip_pitch: geometry 
- link left_hip_roll: geometry 
- link left_hip_yaw: geometry 
- link left_knee: geometry 
- link left_shoulder_pitch: geometry 
- link left_shoulder_roll: geometry 
- link right_ankle_pitch: geometry 
- link right_ankle_roll: geometry 
- link right_elbow: geometry 
- link right_hip_pitch: geometry 
- link right_hip_roll: geometry 
- link right_hip_yaw: geometry 
- link right_knee: geometry 
- link right_shoulder_pitch: geometry 
- link right_shoulder_roll: geometry 
- link trunk: geometry 

Commit message: Model correction (new higher cleats and dxl-64 in neck)

File: common/sigmaban.urdf (robot description, URDF)
Before this commit: robot metabot, 26 links, 25 joints
Joints:
- joint head_pitch: origin xyz=0 0 0.05175 rpy=0 -0 0 -> xyz=0 0 0 rpy=0 -0 0
- joint head_yaw: origin xyz=0.0259 0 0.19943 rpy=0 0 0 -> xyz=0.0259 0 0.268 rpy=0 0 0
- joint left_foot_tip: origin xyz=0 0 -0.05765 rpy=0 0 0 -> xyz=0 0 -0.066 rpy=0 0 0
- joint right_foot_tip: origin xyz=0 0 -0.05765 rpy=0 0 0 -> xyz=0 0 -0.066 rpy=0 0 0

Commit message: Changing camera orientation to match new standard

File: common/sigmaban.urdf (robot description, URDF)
Before this commit: robot metabot, 26 links, 25 joints
Joints:
- joint camera: origin xyz=0.02277 0 0.068925 rpy=0 0 0 -> xyz=0.02277 0 0.068925 rpy=-1.5708 0 -1.5708
